File: FlashlightEagle/Flashlight.brd (EAGLE design)
At the start: 63.5 x 50.5 mm, 29 parts, among them IC1 7805T, T1 BC547, T2 BC547, T3 BC547, X2 Filiament, X3 LED, X4 Switch, X5 Input, X6 Battery

Commit message: Add files via upload
Parts:
- R8: device resistor:R1206 -> resistor:0204/7
- moved C2 2.54 mm to (21.6, 16.5), turned to 270 degrees
- moved C4 1.27 mm to (14.0, 26.7)
- moved R8 1.27 mm to (17.8, 20.3)
Connections:
- removed net N$18: C3.1, X5.1
- net GND: now also C3.1, X5.1
Routing:
- net GND: track 150.5 -> 178.5 mm
- net N$18: track 6.48 -> 0.00 mm
- net N$13: track 24.7 -> 21.9 mm
- net N$15: track 26.7 -> 27.9 mm, vias 0 -> 2
Changed lines of the file:
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@@
 </element>
 <element name="U$2" library="mcp73831" package="SOT23-5L" value="MCP73831" x="17.78" y="27.94" rot="MR0"/>
-<element name="R8" library="resistor" library_urn="urn:adsk.eagle:library:348" package="R1206" package3d_urn="urn:adsk.eagle:package:26062/1" value="" x="17.78" y="21.59" rot="MR90"/>
+<element name="R8" library="resistor" library_urn="urn:adsk.eagle:library:348" package="0204/7" package3d_urn="urn:adsk.eagle:package:25945/1" value="" x="17.78" y="20.32" rot="MR90"/>
 <element name="R9" library="resistor" library_urn="urn:adsk.eagle:library:348" package="R1206" package3d_urn="urn:adsk.eagle:package:26062/1" value="" x="31.75" y="25.4" rot="MR180"/>
 <element name="C1" library="resistor" library_urn="urn:adsk.eagle:library:348" package="C050-025X075" package3d_urn="urn:adsk.eagle:package:26160/1" value="" x="16.51" y="-1.27"/>
-<element name="C2" library="resistor" library_urn="urn:adsk.eagle:library:348" package="C050-025X075" package3d_urn="urn:adsk.eagle:package:26160/1" value="" x="19.05" y="16.51"/>
+<element name="C2" library="resistor" library_urn="urn:adsk.eagle:library:348" package="C050-025X075" package3d_urn="urn:adsk.eagle:package:26160/1" value="" x="21.59" y="16.51" rot="R270"/>
 <element name="C3" library="resistor" library_urn="urn:adsk.eagle:library:348" package="C050-025X075" package3d_urn="urn:adsk.eagle:package:26160/1" value="" x="20.32" y="38.1" rot="R270"/>
-<element name="C4" library="resistor" library_urn="urn:adsk.eagle:library:348" package="C050-025X075" package3d_urn="urn:adsk.eagle:package:26160/1" value="" x="13.97" y="27.94" rot="R90"/>
+<element name="C4" library="resistor" library_urn="urn:adsk.eagle:library:348" package="C050-025X075" package3d_urn="urn:adsk.eagle:package:26160/1" value="" x="13.97" y="26.67" rot="R90"/>
 <element name="X5" library="con-phoenix-254" library_urn="urn:adsk.eagle:library:172" package="2POL254" package3d_urn="urn:adsk.eagle:package:9320/1" value="Input" x="13.97" y="40.64" rot="R270">
 <attribute name="MF" value="" x="13.97" y="40.64" size="1.778" layer="27" rot="R270" display="off"/>
@@
 <wire x1="5.08" y1="29.21" x2="5.08" y2="19.05" width="1.27" layer="16"/>
 <wire x1="5.08" y1="19.05" x2="12.7" y2="19.05" width="1.27" layer="16"/>
-<wire x1="12.7" y1="8.89" x2="12.7" y2="16.51" width="1.27" layer="16"/>
-<wire x1="12.7" y1="16.51" x2="12.7" y2="19.05" width="1.27" layer="16"/>
+<wire x1="12.7" y1="8.89" x2="12.7" y2="19.05" width="1.27" layer="16"/>
 <wire x1="20.32" y1="8.89" x2="12.7" y2="8.89" width="1.27" layer="16"/>
 <wire x1="25.4" y1="5.08" x2="25.4" y2="2.54" width="1.27" layer="16"/>
@@
 <contactref element="C1" pad="1"/>
 <contactref element="C4" pad="1"/>
-<wire x1="16.51" y1="16.51" x2="12.7" y2="16.51" width="1.27" layer="16"/>
 <wire x1="12.7" y1="2.54" x2="12.7" y2="0" width="1.27" layer="16"/>
 <wire x1="12.7" y1="0" x2="13.97" y2="-1.27" width="1.27" layer="16"/>
-<wire x1="17.78" y1="20.168" x2="17.78" y2="17.78" width="1.27" layer="16"/>
-<wire x1="17.78" y1="17.78" x2="16.51" y2="16.51" width="1.27" layer="16"/>
-<wire x1="13.97" y1="25.4" x2="17.78" y2="25.4" width="0.4064" layer="16"/>
+<wire x1="13.97" y1="24.13" x2="17.78" y2="25.4" width="0.4064" layer="16"/>
 <wire x1="17.78" y1="25.4" x2="17.78" y2="26.64" width="0.4064" layer="16"/>
-<wire x1="13.97" y1="25.4" x2="12.7" y2="25.4" width="1.016" layer="16"/>
-<wire x1="12.7" y1="25.4" x2="12.7" y2="22.86" width="1.016" layer="16"/>
+<wire x1="13.97" y1="24.13" x2="12.7" y2="24.13" width="1.016" layer="16"/>
+<wire x1="12.7" y1="24.13" x2="12.7" y2="22.86" width="1.016" layer="16"/>
 <wire x1="12.7" y1="22.86" x2="12.7" y2="19.05" width="1.016" layer="1"/>
 <via x="12.7" y="22.86" extent="1-16" drill="0.35"/>
 <via x="12.7" y="19.05" extent="1-16" drill="0.35"/>
 <contactref element="X6" pad="2"/>
-<wire x1="11.43" y1="34.29" x2="12.562" y2="34.29" width="0.508" layer="16"/>
-<wire x1="12.562" y1="34.29" x2="12.562" y2="31.8804" width="0.508" layer="16"/>
-<wire x1="12.562" y1="31.8804" x2="12.7" y2="31.8804" width="0.508" layer="16"/>
-<wire x1="12.7" y1="31.8804" x2="12.7" y2="25.4" width="0.508" layer="16"/>
+<wire x1="11.292" y1="34.29" x2="11.292" y2="31.8804" width="0.508" layer="16"/>
+<wire x1="11.292" y1="31.8804" x2="12.7" y2="31.8804" width="0.508" layer="16"/>
+<wire x1="12.7" y1="31.8804" x2="12.7" y2="24.13" width="0.508" layer="16"/>
+<contactref element="X5" pad="1"/>
+<contactref element="C3" pad="1"/>
+<wire x1="20.32" y1="40.64" x2="13.97" y2="41.91" width="1.016" layer="16"/>
+<wire x1="13.97" y1="41.91" x2="8.89" y2="41.91" width="0.8128" layer="16"/>
+<wire x1="8.89" y1="34.29" x2="11.292" y2="34.29" width="0.8128" layer="16"/>
+<wire x1="11.292" y1="34.29" x2="11.43" y2="34.29" width="0.8128" layer="16"/>
+<wire x1="8.89" y1="41.91" x2="8.89" y2="34.29" width="0.8128" layer="16"/>
+<wire x1="17.78" y1="16.51" x2="12.7" y2="16.51" width="0.8128" layer="16"/>
+<wire x1="12.7" y1="16.51" x2="12.7" y2="19.05" width="0.8128" layer="16"/>
+<wire x1="21.59" y1="19.05" x2="17.78" y2="19.05" width="0.8128" layer="16"/>
+<wire x1="17.78" y1="19.05" x2="17.78" y2="16.51" width="0.8128" layer="16"/>
 <wire x1="48.1076" y1="15.24" x2="48.26" y2="15.24" width="0" layer="19" extent="16-16"/>
 </signal>
@@
 <wire x1="22.86" y1="8.89" x2="29.21" y2="8.89" width="0.508" layer="16"/>
 <contactref element="C2" pad="2"/>
-<wire x1="20.32" y1="11.43" x2="20.32" y2="15.24" width="1.27" layer="16"/>
-<wire x1="20.32" y1="15.24" x2="21.59" y2="16.51" width="1.27" layer="16"/>
+<wire x1="20.32" y1="11.43" x2="21.59" y2="13.97" width="1.27" layer="16"/>
 </signal>
 <signal name="VCC">
@@
 <wire x1="38.1" y1="13.97" x2="38.1" y2="21.59" width="0.508" layer="16"/>
 <contactref element="X4" pad="1"/>
-<wire x1="20.32" y1="21.59" x2="15.24" y2="21.59" width="0.4064" layer="16"/>
+<wire x1="20.32" y1="21.59" x2="15.24" y2="21.59" width="1.016" layer="16"/>
 <wire x1="38.1" y1="21.59" x2="38.1" y2="29.21" width="1.016" layer="16"/>
 <wire x1="38.1" y1="29.21" x2="31.75" y2="29.21" width="1.016" layer="16"/>
@@
 <wire x1="24.13" y1="29.21" x2="24.13" y2="22.86" width="0.4064" layer="16"/>
 <wire x1="24.13" y1="22.86" x2="21.438" y2="23.012" width="0.4064" layer="16"/>
-<wire x1="21.438" y1="23.012" x2="17.78" y2="23.012" width="0.4064" layer="16"/>
+<wire x1="21.438" y1="23.012" x2="17.78" y2="24.13" width="0.4064" layer="16"/>
 </signal>
 <signal name="N$15">
@@
 <contactref element="U$2" pad="3"/>
 <contactref element="X4" pad="2"/>
-<wire x1="16.8" y1="27.94" x2="13.97" y2="27.94" width="0.4064" layer="16"/>
-<wire x1="13.97" y1="27.94" x2="13.97" y2="30.48" width="0.4064" layer="16"/>
-<wire x1="29.21" y1="29.21" x2="29.21" y2="30.48" width="0.4064" layer="16"/>
-<wire x1="29.21" y1="30.48" x2="17.78" y2="30.48" width="0.4064" layer="16"/>
-<wire x1="17.78" y1="30.48" x2="17.78" y2="27.94" width="0.4064" layer="16"/>
-<wire x1="17.78" y1="27.94" x2="16.8" y2="27.94" width="0.4064" layer="16"/>
 <contactref element="X6" pad="1"/>
-<wire x1="16.83" y1="26.64" x2="16.8" y2="26.64" width="0.508" layer="16"/>
-<wire x1="16.8" y1="26.64" x2="16.8" y2="27.94" width="0.508" layer="16"/>
-<wire x1="13.97" y1="30.48" x2="13.97" y2="34.29" width="0.508" layer="16"/>
-</signal>
-<signal name="N$18">
-<contactref element="X5" pad="1"/>
-<contactref element="C3" pad="1"/>
-<wire x1="20.32" y1="40.64" x2="13.97" y2="41.91" width="1.016" layer="16"/>
+<wire x1="13.97" y1="34.29" x2="13.97" y2="31.75" width="1.27" layer="16"/>
+<wire x1="13.97" y1="31.75" x2="13.97" y2="29.21" width="1.27" layer="16"/>
+<wire x1="29.21" y1="29.21" x2="29.21" y2="31.75" width="1.27" layer="16"/>
+<wire x1="29.21" y1="31.75" x2="19.05" y2="31.75" width="1.27" layer="16"/>
+<wire x1="13.97" y1="31.75" x2="19.05" y2="31.75" width="1.27" layer="1"/>
+<via x="13.97" y="31.75" extent="1-16" drill="0.35"/>
+<via x="19.05" y="31.75" extent="1-16" drill="0.35"/>
+<wire x1="13.97" y1="29.21" x2="13.97" y2="26.67" width="0.4064" layer="16"/>
+<wire x1="13.97" y1="26.67" x2="16.51" y2="26.67" width="0.4064" layer="16"/>
+<wire x1="16.51" y1="26.67" x2="16.83" y2="26.64" width="0" layer="19" extent="16-16"/>
 </signal>
 <signal name="N$19">
@@
 <wire x1="20.32" y1="35.56" x2="20.32" y2="38.1" width="1.016" layer="16"/>
 <wire x1="20.32" y1="38.1" x2="13.97" y2="39.37" width="1.016" layer="16"/>
-<wire x1="20.32" y1="35.56" x2="16.83" y2="35.56" width="1.016" layer="16"/>
-<wire x1="16.83" y1="35.56" x2="16.83" y2="29.24" width="1.016" layer="16"/>
+<wire x1="20.32" y1="35.56" x2="16.83" y2="35.56" width="0.6096" layer="16"/>
+<wire x1="16.83" y1="35.56" x2="16.83" y2="29.24" width="0.6096" layer="16"/>
 <contactref element="R9" pad="2"/>
 <wire x1="33.172" y1="25.4" x2="35.56" y2="25.4" width="0.508" layer="16"/>
