File: FlashlightEagle/Flashlight.sch (EAGLE design)
At the start: 30 parts, among them IC1 7805T, IC2 TP4056, T1 BC547, T2 BC547, T3 BC547, X2 Filiament, X3 LED, X4 Switch, X5 Input

Commit message: Add files via upload
Parts:
- added C1, C2: 3.3µ, resistor:CPOL-EUE2.5-6
- R1, R10, R2, R3: value (none) -> 330R
- R11, R12: value (none) -> 1R
- R4, R5, R6: value (none) -> 8.2K
- R7: value (none) -> 2R
- R8: value (none) -> 1.2R
- R9: value (none) -> 1K
Connections:
- net GND: now also C1.-, C2.-
- net N$13: now also C2.+
- net VCC: now also C1.+
Other:
- moved on the sheet: LED1, LED2, R10, R11, R9, TP1, TP2, X4-1

Commit message: Add files via upload
Parts:
- FILIAMENT: value Filiament -> (none)
- INPUT: value Input -> (none)
- LED: value LED -> (none)
- SWITCH: value Switch -> (none)
- renumbered X2 to FILIAMENT, X3 to LED, X4 to SWITCH, X5 to INPUT
Changed lines of the file:
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@@
 <?xml version="1.0" encoding="utf-8"?>
 <!DOCTYPE eagle SYSTEM "eagle.dtd">
-<eagle version="8.7.1">
+<eagle version="9.0.0">
 <drawing>
 <settings>
@@
 <part name="P+3" library="supply1" library_urn="urn:adsk.eagle:library:371" deviceset="VCC" device=""/>
 <part name="P+4" library="supply1" library_urn="urn:adsk.eagle:library:371" deviceset="VCC" device=""/>
-<part name="X2" library="con-phoenix-254" library_urn="urn:adsk.eagle:library:172" deviceset="MPT2" device="" package3d_urn="urn:adsk.eagle:package:9320/1" value="Filiament"/>
-<part name="X3" library="con-phoenix-254" library_urn="urn:adsk.eagle:library:172" deviceset="MPT2" device="" package3d_urn="urn:adsk.eagle:package:9320/1" value="LED"/>
+<part name="FILIAMENT" library="con-phoenix-254" library_urn="urn:adsk.eagle:library:172" deviceset="MPT2" device="" package3d_urn="urn:adsk.eagle:package:9320/1"/>
+<part name="LED" library="con-phoenix-254" library_urn="urn:adsk.eagle:library:172" deviceset="MPT2" device="" package3d_urn="urn:adsk.eagle:package:9320/1"/>
 <part name="GND6" library="supply1" library_urn="urn:adsk.eagle:library:371" deviceset="GND" device=""/>
 <part name="R7" library="resistor" library_urn="urn:adsk.eagle:library:348" deviceset="R-EU_" device="0411/12" package3d_urn="urn:adsk.eagle:package:26091/1" value="2R"/>
@@
 <part name="GND9" library="supply1" library_urn="urn:adsk.eagle:library:371" deviceset="GND" device=""/>
 <part name="GND10" library="supply1" library_urn="urn:adsk.eagle:library:371" deviceset="GND" device=""/>
-<part name="X5" library="con-phoenix-254" library_urn="urn:adsk.eagle:library:172" deviceset="MPT2" device="" package3d_urn="urn:adsk.eagle:package:9320/1" value="Input"/>
+<part name="INPUT" library="con-phoenix-254" library_urn="urn:adsk.eagle:library:172" deviceset="MPT2" device="" package3d_urn="urn:adsk.eagle:package:9320/1"/>
 <part name="GND11" library="supply1" library_urn="urn:adsk.eagle:library:371" deviceset="GND" device=""/>
 <part name="LED1" library="led" library_urn="urn:adsk.eagle:library:259" deviceset="LED" device="3MM" package3d_urn="urn:adsk.eagle:package:15797/1"/>
@@
 <part name="TP1" library="testpad" library_urn="urn:adsk.eagle:library:385" deviceset="PTR1" device="PAD1-13" package3d_urn="urn:adsk.eagle:package:27946/1" value="PTR1PAD1-13"/>
 <part name="TP2" library="testpad" library_urn="urn:adsk.eagle:library:385" deviceset="PTR1" device="PAD1-13" package3d_urn="urn:adsk.eagle:package:27946/1" value="PTR1PAD1-13"/>
-<part name="X4" library="con-phoenix-254" library_urn="urn:adsk.eagle:library:172" deviceset="MPT2" device="" package3d_urn="urn:adsk.eagle:package:9320/1" value="Switch"/>
+<part name="SWITCH" library="con-phoenix-254" library_urn="urn:adsk.eagle:library:172" deviceset="MPT2" device="" package3d_urn="urn:adsk.eagle:package:9320/1"/>
 <part name="C1" library="resistor" library_urn="urn:adsk.eagle:library:348" deviceset="CPOL-EU" device="E2.5-6" package3d_urn="urn:adsk.eagle:package:25832/1" value="3.3µ"/>
 <part name="C2" library="resistor" library_urn="urn:adsk.eagle:library:348" deviceset="CPOL-EU" device="E2.5-6" package3d_urn="urn:adsk.eagle:package:25832/1" value="3.3µ"/>
@@
 <instance part="P+3" gate="VCC" x="106.68" y="71.12" rot="R270"/>
 <instance part="P+4" gate="VCC" x="106.68" y="53.34" rot="R270"/>
-<instance part="X2" gate="-1" x="-91.44" y="63.5" rot="R180"/>
-<instance part="X2" gate="-2" x="-91.44" y="73.66" rot="R180"/>
-<instance part="X3" gate="-1" x="-45.72" y="58.42" rot="R270"/>
-<instance part="X3" gate="-2" x="-83.82" y="66.04" rot="R90"/>
+<instance part="FILIAMENT" gate="-1" x="-91.44" y="63.5" rot="R180"/>
+<instance part="FILIAMENT" gate="-2" x="-91.44" y="73.66" rot="R180"/>
+<instance part="LED" gate="-1" x="-45.72" y="58.42" rot="R270"/>
+<instance part="LED" gate="-2" x="-83.82" y="66.04" rot="R90"/>
 <instance part="GND6" gate="1" x="-83.82" y="60.96"/>
 <instance part="R7" gate="G$1" x="-45.72" y="66.04" rot="R90"/>
@@
 <instance part="GND9" gate="1" x="63.5" y="-5.08"/>
 <instance part="GND10" gate="1" x="-20.32" y="27.94" rot="R270"/>
-<instance part="X5" gate="-1" x="-58.42" y="15.24" rot="R180"/>
-<instance part="X5" gate="-2" x="-58.42" y="20.32" rot="R180"/>
+<instance part="INPUT" gate="-1" x="-58.42" y="15.24" rot="R180"/>
+<instance part="INPUT" gate="-2" x="-58.42" y="20.32" rot="R180"/>
 <instance part="GND11" gate="1" x="-55.88" y="12.7"/>
 <instance part="LED1" gate="G$1" x="60.96" y="27.94" rot="R270"/>
@@
 <instance part="TP1" gate="G$1" x="43.18" y="20.32" rot="R90"/>
 <instance part="TP2" gate="G$1" x="71.12" y="-2.54" rot="R90"/>
-<instance part="X4" gate="-1" x="38.1" y="17.78" rot="R180"/>
-<instance part="X4" gate="-2" x="-66.04" y="83.82" rot="R270"/>
+<instance part="SWITCH" gate="-1" x="38.1" y="17.78" rot="R180"/>
+<instance part="SWITCH" gate="-2" x="-66.04" y="83.82" rot="R270"/>
 <instance part="C1" gate="G$1" x="-38.1" y="60.96"/>
 <instance part="C2" gate="G$1" x="-15.24" y="60.96"/>
@@
 <pinref part="PAD3" gate="1" pin="P"/>
 <wire x1="-78.74" y1="63.5" x2="-83.82" y2="63.5" width="0.1524" layer="91"/>
-<pinref part="X2" gate="-1" pin="1"/>
-<pinref part="X3" gate="-2" pin="1"/>
+<pinref part="FILIAMENT" gate="-1" pin="1"/>
+<pinref part="LED" gate="-2" pin="1"/>
 <wire x1="-83.82" y1="63.5" x2="-88.9" y2="63.5" width="0.1524" layer="91"/>
 <junction x="-83.82" y="63.5"/>
@@
 </segment>
 <segment>
-<pinref part="X5" gate="-1" pin="1"/>
+<pinref part="INPUT" gate="-1" pin="1"/>
 <pinref part="GND11" gate="1" pin="GND"/>
 </segment>
@@
 <pinref part="C2" gate="G$1" pin="+"/>
 <junction x="-15.24" y="63.5"/>
+<junction x="-5.08" y="63.5"/>
 </segment>
 </net>
@@
 <junction x="-38.1" y="63.5"/>
 <wire x1="-38.1" y1="63.5" x2="-35.56" y2="63.5" width="0.1524" layer="91"/>
+<junction x="-38.1" y="71.12"/>
 </segment>
 <segment>
@@
 <wire x1="-78.74" y1="86.36" x2="-78.74" y2="73.66" width="0.1524" layer="91"/>
 <wire x1="-78.74" y1="73.66" x2="-88.9" y2="73.66" width="0.1524" layer="91"/>
-<pinref part="X2" gate="-2" pin="1"/>
+<pinref part="FILIAMENT" gate="-2" pin="1"/>
 <junction x="-78.74" y="73.66"/>
-<pinref part="X4" gate="-2" pin="1"/>
+<pinref part="SWITCH" gate="-2" pin="1"/>
 <junction x="-66.04" y="86.36"/>
 </segment>
@@
 <segment>
 <pinref part="R7" gate="G$1" pin="1"/>
-<pinref part="X3" gate="-1" pin="1"/>
+<pinref part="LED" gate="-1" pin="1"/>
 </segment>
 </net>
@@
 <pinref part="T1" gate="G$1" pin="C"/>
 <wire x1="83.82" y1="88.9" x2="71.12" y2="88.9" width="0.1524" layer="91"/>
+<junction x="83.82" y="88.9"/>
 </segment>
 </net>
@@
 <pinref part="T2" gate="G$1" pin="C"/>
 <wire x1="83.82" y1="71.12" x2="71.12" y2="71.12" width="0.1524" layer="91"/>
+<junction x="83.82" y="71.12"/>
 </segment>
 </net>
@@
 <wire x1="27.94" y1="22.86" x2="40.64" y2="20.32" width="0.1524" layer="91"/>
 <pinref part="TP1" gate="G$1" pin="TP"/>
-<pinref part="X4" gate="-1" pin="1"/>
+<pinref part="SWITCH" gate="-1" pin="1"/>
 <junction x="40.64" y="20.32"/>
 <wire x1="40.64" y1="20.32" x2="40.64" y2="17.78" width="0.1524" layer="91"/>
@@
 <pinref part="R12" gate="G$1" pin="1"/>
 <wire x1="-7.62" y1="5.08" x2="-2.54" y2="5.08" width="0.1524" layer="91"/>
-<pinref part="X5" gate="-2" pin="1"/>
+<pinref part="INPUT" gate="-2" pin="1"/>
 <wire x1="-2.54" y1="5.08" x2="0" y2="5.08" width="0.1524" layer="91"/>
 <wire x1="-55.88" y1="20.32" x2="-20.32" y2="20.32" width="0.1524" layer="91"/>

Commit message: Add files via upload
Parts:
- X2: value (none) -> Filiament
- X3: value (none) -> LED
- X4: value (none) -> Switch
- X5: value (none) -> Input
- renumbered FILIAMENT to X2, INPUT to X5, LED to X3, SWITCH to X4
Changed lines of the file:
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@@
 <?xml version="1.0" encoding="utf-8"?>
 <!DOCTYPE eagle SYSTEM "eagle.dtd">
-<eagle version="9.0.0">
+<eagle version="9.1.1">
 <drawing>
 <settings>
@@
 <part name="P+3" library="supply1" library_urn="urn:adsk.eagle:library:371" deviceset="VCC" device=""/>
 <part name="P+4" library="supply1" library_urn="urn:adsk.eagle:library:371" deviceset="VCC" device=""/>
-<part name="FILIAMENT" library="con-phoenix-254" library_urn="urn:adsk.eagle:library:172" deviceset="MPT2" device="" package3d_urn="urn:adsk.eagle:package:9320/1"/>
-<part name="LED" library="con-phoenix-254" library_urn="urn:adsk.eagle:library:172" deviceset="MPT2" device="" package3d_urn="urn:adsk.eagle:package:9320/1"/>
+<part name="X2" library="con-phoenix-254" library_urn="urn:adsk.eagle:library:172" deviceset="MPT2" device="" package3d_urn="urn:adsk.eagle:package:9320/1" value="Filiament"/>
+<part name="X3" library="con-phoenix-254" library_urn="urn:adsk.eagle:library:172" deviceset="MPT2" device="" package3d_urn="urn:adsk.eagle:package:9320/1" value="LED"/>
 <part name="GND6" library="supply1" library_urn="urn:adsk.eagle:library:371" deviceset="GND" device=""/>
 <part name="R7" library="resistor" library_urn="urn:adsk.eagle:library:348" deviceset="R-EU_" device="0411/12" package3d_urn="urn:adsk.eagle:package:26091/1" value="2R"/>
@@
 <part name="GND9" library="supply1" library_urn="urn:adsk.eagle:library:371" deviceset="GND" device=""/>
 <part name="GND10" library="supply1" library_urn="urn:adsk.eagle:library:371" deviceset="GND" device=""/>
-<part name="INPUT" library="con-phoenix-254" library_urn="urn:adsk.eagle:library:172" deviceset="MPT2" device="" package3d_urn="urn:adsk.eagle:package:9320/1"/>
+<part name="X5" library="con-phoenix-254" library_urn="urn:adsk.eagle:library:172" deviceset="MPT2" device="" package3d_urn="urn:adsk.eagle:package:9320/1" value="Input"/>
 <part name="GND11" library="supply1" library_urn="urn:adsk.eagle:library:371" deviceset="GND" device=""/>
 <part name="LED1" library="led" library_urn="urn:adsk.eagle:library:259" deviceset="LED" device="3MM" package3d_urn="urn:adsk.eagle:package:15797/1"/>
@@
 <part name="TP1" library="testpad" library_urn="urn:adsk.eagle:library:385" deviceset="PTR1" device="PAD1-13" package3d_urn="urn:adsk.eagle:package:27946/1" value="PTR1PAD1-13"/>
 <part name="TP2" library="testpad" library_urn="urn:adsk.eagle:library:385" deviceset="PTR1" device="PAD1-13" package3d_urn="urn:adsk.eagle:package:27946/1" value="PTR1PAD1-13"/>
-<part name="SWITCH" library="con-phoenix-254" library_urn="urn:adsk.eagle:library:172" deviceset="MPT2" device="" package3d_urn="urn:adsk.eagle:package:9320/1"/>
+<part name="X4" library="con-phoenix-254" library_urn="urn:adsk.eagle:library:172" deviceset="MPT2" device="" package3d_urn="urn:adsk.eagle:package:9320/1" value="Switch"/>
 <part name="C1" library="resistor" library_urn="urn:adsk.eagle:library:348" deviceset="CPOL-EU" device="E2.5-6" package3d_urn="urn:adsk.eagle:package:25832/1" value="3.3µ"/>
 <part name="C2" library="resistor" library_urn="urn:adsk.eagle:library:348" deviceset="CPOL-EU" device="E2.5-6" package3d_urn="urn:adsk.eagle:package:25832/1" value="3.3µ"/>
@@
 <instance part="P+3" gate="VCC" x="106.68" y="71.12" rot="R270"/>
 <instance part="P+4" gate="VCC" x="106.68" y="53.34" rot="R270"/>
-<instance part="FILIAMENT" gate="-1" x="-91.44" y="63.5" rot="R180"/>
-<instance part="FILIAMENT" gate="-2" x="-91.44" y="73.66" rot="R180"/>
-<instance part="LED" gate="-1" x="-45.72" y="58.42" rot="R270"/>
-<instance part="LED" gate="-2" x="-83.82" y="66.04" rot="R90"/>
+<instance part="X2" gate="-1" x="-91.44" y="63.5" rot="R180"/>
+<instance part="X2" gate="-2" x="-91.44" y="73.66" rot="R180"/>
+<instance part="X3" gate="-1" x="-45.72" y="58.42" rot="R270"/>
+<instance part="X3" gate="-2" x="-83.82" y="66.04" rot="R90"/>
 <instance part="GND6" gate="1" x="-83.82" y="60.96"/>
 <instance part="R7" gate="G$1" x="-45.72" y="66.04" rot="R90"/>
@@
 <instance part="GND9" gate="1" x="63.5" y="-5.08"/>
 <instance part="GND10" gate="1" x="-20.32" y="27.94" rot="R270"/>
-<instance part="INPUT" gate="-1" x="-58.42" y="15.24" rot="R180"/>
-<instance part="INPUT" gate="-2" x="-58.42" y="20.32" rot="R180"/>
+<instance part="X5" gate="-1" x="-58.42" y="15.24" rot="R180"/>
+<instance part="X5" gate="-2" x="-58.42" y="20.32" rot="R180"/>
 <instance part="GND11" gate="1" x="-55.88" y="12.7"/>
 <instance part="LED1" gate="G$1" x="60.96" y="27.94" rot="R270"/>
@@
 <instance part="TP1" gate="G$1" x="43.18" y="20.32" rot="R90"/>
 <instance part="TP2" gate="G$1" x="71.12" y="-2.54" rot="R90"/>
-<instance part="SWITCH" gate="-1" x="38.1" y="17.78" rot="R180"/>
-<instance part="SWITCH" gate="-2" x="-66.04" y="83.82" rot="R270"/>
+<instance part="X4" gate="-1" x="38.1" y="17.78" rot="R180"/>
+<instance part="X4" gate="-2" x="-66.04" y="83.82" rot="R270"/>
 <instance part="C1" gate="G$1" x="-38.1" y="60.96"/>
 <instance part="C2" gate="G$1" x="-15.24" y="60.96"/>
@@
 <pinref part="PAD3" gate="1" pin="P"/>
 <wire x1="-78.74" y1="63.5" x2="-83.82" y2="63.5" width="0.1524" layer="91"/>
-<pinref part="FILIAMENT" gate="-1" pin="1"/>
-<pinref part="LED" gate="-2" pin="1"/>
+<pinref part="X2" gate="-1" pin="1"/>
+<pinref part="X3" gate="-2" pin="1"/>
 <wire x1="-83.82" y1="63.5" x2="-88.9" y2="63.5" width="0.1524" layer="91"/>
 <junction x="-83.82" y="63.5"/>
@@
 </segment>
 <segment>
-<pinref part="INPUT" gate="-1" pin="1"/>
+<pinref part="X5" gate="-1" pin="1"/>
 <pinref part="GND11" gate="1" pin="GND"/>
 </segment>
@@
 <pinref part="C2" gate="G$1" pin="+"/>
 <junction x="-15.24" y="63.5"/>
-<junction x="-5.08" y="63.5"/>
 </segment>
 </net>
@@
 <junction x="-38.1" y="63.5"/>
 <wire x1="-38.1" y1="63.5" x2="-35.56" y2="63.5" width="0.1524" layer="91"/>
-<junction x="-38.1" y="71.12"/>
 </segment>
 <segment>
@@
 <wire x1="-78.74" y1="86.36" x2="-78.74" y2="73.66" width="0.1524" layer="91"/>
 <wire x1="-78.74" y1="73.66" x2="-88.9" y2="73.66" width="0.1524" layer="91"/>
-<pinref part="FILIAMENT" gate="-2" pin="1"/>
+<pinref part="X2" gate="-2" pin="1"/>
 <junction x="-78.74" y="73.66"/>
-<pinref part="SWITCH" gate="-2" pin="1"/>
+<pinref part="X4" gate="-2" pin="1"/>
 <junction x="-66.04" y="86.36"/>
 </segment>
@@
 <segment>
 <pinref part="R7" gate="G$1" pin="1"/>
-<pinref part="LED" gate="-1" pin="1"/>
+<pinref part="X3" gate="-1" pin="1"/>
 </segment>
 </net>
@@
 <pinref part="T1" gate="G$1" pin="C"/>
 <wire x1="83.82" y1="88.9" x2="71.12" y2="88.9" width="0.1524" layer="91"/>
-<junction x="83.82" y="88.9"/>
 </segment>
 </net>
@@
 <pinref part="T2" gate="G$1" pin="C"/>
 <wire x1="83.82" y1="71.12" x2="71.12" y2="71.12" width="0.1524" layer="91"/>
-<junction x="83.82" y="71.12"/>
 </segment>
 </net>
@@
 <wire x1="27.94" y1="22.86" x2="40.64" y2="20.32" width="0.1524" layer="91"/>
 <pinref part="TP1" gate="G$1" pin="TP"/>
-<pinref part="SWITCH" gate="-1" pin="1"/>
+<pinref part="X4" gate="-1" pin="1"/>
 <junction x="40.64" y="20.32"/>
 <wire x1="40.64" y1="20.32" x2="40.64" y2="17.78" width="0.1524" layer="91"/>
@@
 <pinref part="R12" gate="G$1" pin="1"/>
 <wire x1="-7.62" y1="5.08" x2="-2.54" y2="5.08" width="0.1524" layer="91"/>
-<pinref part="INPUT" gate="-2" pin="1"/>
+<pinref part="X5" gate="-2" pin="1"/>
 <wire x1="-2.54" y1="5.08" x2="0" y2="5.08" width="0.1524" layer="91"/>
 <wire x1="-55.88" y1="20.32" x2="-20.32" y2="20.32" width="0.1524" layer="91"/>
